File: Light_controller.sch (KiCad schematic (older format))
At the start: 42 parts, among them U1 LM358, U10 PH2.0_horizontal, U11 PH2.0_horizontal, U12 PH2.0_horizontal, U2 PT8211-S, U3 STM8S003F3P, U4 SMD_2062, U5 tact_sw, U6 AMS1117-5.0, U7 EL357N-C, U8 EL357N-C, U9 PH2.0_horizontal

Commit message: modified layout but havent fill ground yet
Parts:
- removed D? (x2): D_Zener, symbol Device:D_Zener
- added D2, D3: BZX84Cxx, Diode_SMD:D_SOT-23_ANK, symbol Diode:BZX84Cxx
- JP1: renamed from JP?; footprint (none) -> Jumper:SolderJumper-2_P1.3mm_Open_TrianglePad1.0x1.5mm
- U13: renamed from U?; footprint (none) -> Custom_footprint_lib:custom_pinsocket_1x04_p2.54
- U14: renamed from U?; footprint (none) -> Custom_footprint_lib:SMD2063
- gave numbers to parts that had none: 5
Connections:
- net labels removed: PA1, PA2, PA3, PB5, PC4, PC7, UART_CLOCK, VCAP
- wire segments 136 -> 132
Changed lines of the file:
@@
 $EndComp
-Wire Wire Line
-	10600 1900 11100 1900
 Wire Wire Line
 	10600 2000 11100 2000
 Wire Wire Line
 	10600 2100 11100 2100
-Text Label 10650 1900 0    50   ~ 0
-UART_CLOCK
 Text Label 10800 2000 0    50   ~ 0
 UART_TX
@@
 	10600 1800 11100 1800
 Wire Wire Line
-	10600 1700 11100 1700
-Wire Wire Line
 	10600 1600 11100 1600
 Wire Wire Line
-	8900 1200 9400 1200
-Wire Wire Line
-	8900 1300 9400 1300
-Wire Wire Line
-	8900 1400 9400 1400
-Wire Wire Line
-	8900 1700 9400 1700
-Wire Wire Line
 	8900 1600 9400 1600
-Wire Wire Line
-	8900 2300 9400 2300
-Wire Wire Line
-	8900 1900 9400 1900
 Wire Wire Line
 	8900 2100 9400 2100
@@
 Wire Wire Line
 	1450 4950 1450 4850
-Text Label 8900 1200 0    50   ~ 0
-PA1
-Text Label 8900 1300 0    50   ~ 0
-PA2
-Text Label 8900 1400 0    50   ~ 0
-PA3
 Text Label 8900 1600 0    50   ~ 0
 C_SENSOR
-Text Label 8900 1700 0    50   ~ 0
-PB5
-Text Label 8900 1900 0    50   ~ 0
-WS
-Text Label 8900 2300 0    50   ~ 0
-PC7
 Wire Wire Line
 	9400 2500 8900 2500
-Wire Wire Line
-	9400 2600 8900 2600
 Text Notes 550  4200 0    118  ~ 0
 Reset Circuit
 Text Label 8900 2500 0    50   ~ 0
 RESET
-Text Label 8900 2600 0    50   ~ 0
-VCAP
-Text Label 10600 1700 0    50   ~ 0
-TEMP_SENSOR
 Text Label 10750 1800 0    50   ~ 0
 V_SENSOR
@@
 	1    0    0    1
 $EndComp
-Text Label 8900 2000 0    50   ~ 0
-PC4
-Wire Wire Line
-	8900 2000 9400 2000
 Wire Wire Line
 	3750 7000 3750 7050
@@
 Wire Wire Line
 	6150 5900 6150 6450
-Text Label 3600 5900 0    50   ~ 0
+Text Label 4050 5900 2    50   ~ 0
 5V_SUPPLY
 $Comp
@@
 $EndComp
 Wire Wire Line
-	3600 5900 4100 5900
+	3600 5900 4050 5900
 $Comp
 L Custom_Library:EL357N-C U7
@@
 	9650 4950 9550 4950
 Wire Wire Line
-	1900 6200 2150 6200
-Text Label 2150 6200 0    50   ~ 0
+	1900 6200 2000 6200
+Text Label 2000 6200 0    50   ~ 0
 12V_INPUT
 Wire Wire Line
@@
 	7850 5450 7850 5700
 $Comp
-L Custom_Library:SMD2063 U?
+L Custom_Library:SMD2063 U14
 U 1 1 5E8C06BF
 P 10350 4450
-F 0 "U?" H 10350 3700 50  0000 R CNN
+F 0 "U14" H 10350 3700 50  0000 R CNN
 F 1 "SMD2063" H 10500 3800 50  0000 R CNN
-F 2 "" H 10350 4450 50  0001 C CNN
+F 2 "Custom_footprint_lib:SMD2063" H 10350 4450 50  0001 C CNN
 F 3 "" H 10350 4450 50  0001 C CNN
 	1    10350 4450
@@
 Voltage and current for sensor
 $Comp
-L Device:R R?
+L Device:R R13
 U 1 1 5E8FADD1
 P 4750 3200
-F 0 "R?" V 4543 3200 50  0000 C CNN
+F 0 "R13" V 4543 3200 50  0000 C CNN
 F 1 "R" V 4634 3200 50  0000 C CNN
 F 2 "Resistor_SMD:R_0603_1608Metric" V 4680 3200 50  0001 C CNN
@@
 	4750 3050 5150 3050
 $Comp
-L Device:R R?
+L Device:R R14
 U 1 1 5E90AFB8
 P 4750 3900
-F 0 "R?" V 4543 3900 50  0000 C CNN
+F 0 "R14" V 4543 3900 50  0000 C CNN
 F 1 "R" V 4634 3900 50  0000 C CNN
 F 2 "Resistor_SMD:R_0603_1608Metric" V 4680 3900 50  0001 C CNN
@@
 Text Notes 5300 3500 0    50   ~ 0
 (0 to 5V)\n
-$Comp
-L Device:D_Zener D?
-U 1 1 5E929C56
-P 4400 3900
-F 0 "D?" V 4350 3700 50  0000 L CNN
-F 1 "D_Zener" V 4450 3500 50  0000 L CNN
-F 2 "" H 4400 3900 50  0001 C CNN
-F 3 "~" H 4400 3900 50  0001 C CNN
-	1    4400 3900
-	0    1    1    0
-$EndComp
 Wire Wire Line
 	4400 4050 4750 4050
@@
 Text Label 5700 2250 2    50   ~ 0
 LED-
-$Comp
-L Device:D_Zener D?
-U 1 1 5E95453B
-P 4250 1550
-F 0 "D?" V 4200 1350 50  0000 L CNN
-F 1 "D_Zener" V 4300 1150 50  0000 L CNN
-F 2 "" H 4250 1550 50  0001 C CNN
-F 3 "~" H 4250 1550 50  0001 C CNN
-	1    4250 1550
-	0    1    1    0
-$EndComp
 Text Label 3700 1400 0    50   ~ 0
 C_SENSOR
 Connection ~ 4650 1400
 Wire Wire Line
-	3700 1400 4250 1400
-Connection ~ 4250 1400
-Wire Wire Line
-	4250 1400 4650 1400
-Wire Wire Line
 	4250 1700 4250 2000
 Text Label 4250 2000 1    50   ~ 0
 LED-
 $Comp
-L Custom_Library:PinSocket_1x4 U?
+L Custom_Library:PinSocket_1x4 U13
 U 1 1 5E9927B0
 P 7600 4500
-F 0 "U?" H 7800 3550 50  0000 R CNN
+F 0 "U13" H 7800 3550 50  0000 R CNN
 F 1 "PinSocket_1x4" H 7800 3650 50  0000 R CNN
-F 2 "" H 7600 4500 50  0001 C CNN
+F 2 "Custom_footprint_lib:custom_pinsocket_1x04_p2.54" H 7600 4500 50  0001 C CNN
 F 3 "" H 7600 4500 50  0001 C CNN
 	1    7600 4500
@@
 RESET
 $Comp
-L Jumper:SolderJumper_2_Open JP?
-U 1 1 5E9DBABF
-P 7750 2200
-F 0 "JP?" H 7750 2405 50  0000 C CNN
-F 1 "SolderJumper_2_Open" H 7750 2314 50  0000 C CNN
-F 2 "" H 7750 2200 50  0001 C CNN
-F 3 "~" H 7750 2200 50  0001 C CNN
-	1    7750 2200
-	1    0    0    -1
-$EndComp
-Text Label 7200 2200 0    50   ~ 0
-LED-
-Wire Wire Line
-	7200 2200 7600 2200
-$Comp
-L power:GND #PWR?
+L power:GND #PWR0103
 U 1 1 5E9FD433
 P 6950 3950
-F 0 "#PWR?" H 6950 3700 50  0001 C CNN
+F 0 "#PWR0103" H 6950 3700 50  0001 C CNN
 F 1 "GND" H 6955 3777 50  0000 C CNN
 F 2 "" H 6950 3950 50  0001 C CNN
@@
 	6900 4250 7300 4250
 $Comp
-L Device:C C?
+L Device:C C10
 U 1 1 5EA22692
 P 10600 1000
-F 0 "C?" H 10715 1046 50  0000 L CNN
+F 0 "C10" H 10715 1046 50  0000 L CNN
 F 1 "C" H 10715 955 50  0000 L CNN
 F 2 "Capacitor_SMD:C_0805_2012Metric" H 10638 850 50  0001 C CNN
@@
 Connection ~ 10600 850
 $Comp
-L Device:C C?
+L Device:C C9
 U 1 1 5EA39C76
 P 4050 5750
-F 0 "C?" V 4200 5850 50  0000 C CNN
+F 0 "C9" V 4200 5850 50  0000 C CNN
 F 1 "C" V 4200 5750 50  0000 C CNN
 F 2 "Capacitor_SMD:C_0805_2012Metric" H 4088 5600 50  0001 C CNN
@@
 $EndComp
 $Comp
-L power:GND #PWR?
+L power:GND #PWR0104
 U 1 1 5EA3F7D4
 P 3950 5600
-F 0 "#PWR?" H 3950 5350 50  0001 C CNN
+F 0 "#PWR0104" H 3950 5350 50  0001 C CNN
 F 1 "GND" H 3955 5427 50  0000 C CNN
 F 2 "" H 3950 5600 50  0001 C CNN
@@
 	2000 6350 2000 6200
 $Comp
-L Device:C C?
+L Device:C C8
 U 1 1 5EA4B159
 P 2000 6500
-F 0 "C?" V 2150 6600 50  0000 C CNN
+F 0 "C8" V 2150 6600 50  0000 C CNN
 F 1 "C" V 2150 6500 50  0000 C CNN
 F 2 "Capacitor_SMD:C_0805_2012Metric" H 2038 6350 50  0001 C CNN
@@
 $EndComp
 $Comp
-L power:GND #PWR?
+L power:GND #PWR0107
 U 1 1 5EA50995
 P 2000 6750
-F 0 "#PWR?" H 2000 6500 50  0001 C CNN
+F 0 "#PWR0107" H 2000 6500 50  0001 C CNN
 F 1 "GND" H 2005 6577 50  0000 C CNN
 F 2 "" H 2000 6750 50  0001 C CNN
@@
 Wire Wire Line
 	2000 6650 2000 6750
+Wire Wire Line
+	8900 1700 9400 1700
+Text Label 8900 1700 0    50   ~ 0
+TEMP_SENSOR
+Text Label 8900 1900 0    50   ~ 0
+WS
+Wire Wire Line
+	8900 1900 9400 1900
+$Comp
+L Diode:BZX84Cxx D2
+U 1 1 5E80DF83
+P 4250 1550
+F 0 "D2" V 4204 1629 50  0000 L CNN
+F 1 "BZX84Cxx" V 4295 1629 50  0000 L CNN
+F 2 "Diode_SMD:D_SOT-23_ANK" H 4250 1375 50  0001 C CNN
+F 3 "https://diotec.com/tl_files/diotec/files/pdf/datasheets/bzx84c2v4.pdf" H 4250 1550 50  0001 C CNN
+	1    4250 1550
+	0    1    1    0
+$EndComp
+Wire Wire Line
+	3700 1400 4250 1400
+Connection ~ 4250 1400
+Wire Wire Line
+	4250 1400 4650 1400
+$Comp
+L Diode:BZX84Cxx D3
+U 1 1 5E8143F1
+P 4400 3900
+F 0 "D3" V 4350 3600 50  0000 L CNN
+F 1 "BZX84Cxx" V 4450 3450 50  0000 L CNN
+F 2 "Diode_SMD:D_SOT-23_ANK" H 4400 3725 50  0001 C CNN
+F 3 "https://diotec.com/tl_files/diotec/files/pdf/datasheets/bzx84c2v4.pdf" H 4400 3900 50  0001 C CNN
+	1    4400 3900
+	0    1    1    0
+$EndComp
+Wire Wire Line
+	7700 3350 7800 3350
+$Comp
+L power:GND #PWR0108
+U 1 1 5E7CE938
+P 7800 3350
+F 0 "#PWR0108" H 7800 3100 50  0001 C CNN
+F 1 "GND" H 7805 3177 50  0000 C CNN
+F 2 "" H 7800 3350 50  0001 C CNN
+F 3 "" H 7800 3350 50  0001 C CNN
+	1    7800 3350
+	0    -1   -1   0
+$EndComp
+Wire Wire Line
+	7000 3350 7400 3350
+Text Label 7000 3350 0    50   ~ 0
+LED-
+$Comp
+L Jumper:SolderJumper_2_Open JP1
+U 1 1 5E9DBABF
+P 7550 3350
+F 0 "JP1" H 7550 3555 50  0000 C CNN
+F 1 "SolderJumper_2_Open" H 7550 3464 50  0000 C CNN
+F 2 "Jumper:SolderJumper-2_P1.3mm_Open_TrianglePad1.0x1.5mm" H 7550 3350 50  0001 C CNN
+F 3 "~" H 7550 3350 50  0001 C CNN
+	1    7550 3350
+	1    0    0    -1
+$EndComp
+$Comp
+L power:GND #PWR0109
+U 1 1 5E834D03
+P 10600 1200
+F 0 "#PWR0109" H 10600 950 50  0001 C CNN
+F 1 "GND" H 10605 1027 50  0000 C CNN
+F 2 "" H 10600 1200 50  0001 C CNN
+F 3 "" H 10600 1200 50  0001 C CNN
+	1    10600 1200
+	1    0    0    -1
+$EndComp
+Wire Wire Line
+	10600 1150 10600 1200
+Connection ~ 2000 6200
+Wire Wire Line
+	2000 6200 2150 6200
+Connection ~ 4050 5900
+Wire Wire Line
+	4050 5900 4100 5900
 $EndSCHEMATC

Commit message: updated the layout
Parts:
- removed JP1: SolderJumper_2_Open, Jumper:SolderJumper-2_P1.3mm_Open_TrianglePad1.0x1.5mm, symbol Jumper:SolderJumper_2_Open
- added JP1: Jumper_2_Open, Jumper:SolderJumper-2_P1.3mm_Open_TrianglePad1.0x1.5mm, symbol Jumper:Jumper_2_Open
Changed lines of the file:
@@
 	-1   0    0    1
 $EndComp
+Text Label 9600 4250 0    50   ~ 0
+LED-
 Text Label 9600 3950 0    50   ~ 0
-LED-
-Text Label 9600 4250 0    50   ~ 0
 LED+
 Text Label 9600 4100 0    50   ~ 0
@@
 	9600 4100 10000 4100
 Wire Wire Line
+	9600 3950 10000 3950
+Wire Wire Line
 	9600 4250 10000 4250
-Wire Wire Line
-	9600 3950 10000 3950
 Wire Wire Line
 	6100 1700 6100 2000
@@
 Text Notes 5250 3050 0    50   ~ 0
 max 80V
-Text Notes 9200 4250 0    50   ~ 0
+Text Notes 9200 3950 0    50   ~ 0
 max 80V
 Text Notes 5300 3500 0    50   ~ 0
@@
 	0    1    1    0
 $EndComp
-Wire Wire Line
-	7700 3350 7800 3350
 $Comp
 L power:GND #PWR0108
@@
 $EndComp
 Wire Wire Line
-	7000 3350 7400 3350
+	7000 3350 7350 3350
 Text Label 7000 3350 0    50   ~ 0
 LED-
-$Comp
-L Jumper:SolderJumper_2_Open JP1
-U 1 1 5E9DBABF
-P 7550 3350
-F 0 "JP1" H 7550 3555 50  0000 C CNN
-F 1 "SolderJumper_2_Open" H 7550 3464 50  0000 C CNN
-F 2 "Jumper:SolderJumper-2_P1.3mm_Open_TrianglePad1.0x1.5mm" H 7550 3350 50  0001 C CNN
-F 3 "~" H 7550 3350 50  0001 C CNN
-	1    7550 3350
-	1    0    0    -1
-$EndComp
 $Comp
 L power:GND #PWR0109
@@
 Wire Wire Line
 	4050 5900 4100 5900
+Wire Wire Line
+	7750 3350 7800 3350
+$Comp
+L Jumper:Jumper_2_Open JP1
+U 1 1 5E84B2E4
+P 7550 3350
+F 0 "JP1" H 7550 3585 50  0000 C CNN
+F 1 "Jumper_2_Open" H 7550 3494 50  0000 C CNN
+F 2 "Jumper:SolderJumper-2_P1.3mm_Open_TrianglePad1.0x1.5mm" H 7550 3350 50  0001 C CNN
+F 3 "~" H 7550 3350 50  0001 C CNN
+	1    7550 3350
+	1    0    0    -1
+$EndComp
 $EndSCHEMATC
