File: Light_controller.sch (KiCad schematic (older format))
At the start: 44 parts, among them U1 LM358, U10 PH2.0_horizontal, U11 PH2.0_horizontal, U12 PH2.0_horizontal, U13 PinSocket_1x4, U3 STM8S003F3P, U4 SMD_2062, U5 tact_sw, U6 AMS1117-5.0, U7 EL357N-C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

Commit message: added esp32,stm32 circuit
Parts:
- removed D1: 1N5819HW, Diode_SMD:D_SOD-123, symbol Diode:1N5819
- removed D?: BZX84Cxx, Diode_SMD:D_SOT-23_ANK, symbol Diode:BZX84Cxx
- added C?: C, symbol Device:C
- added D?: D_Schottky, symbol Device:D_Schottky
- added R?: R, Resistor_SMD:R_0603_1608Metric, symbol Device:R
- added R?: 2k, Resistor_SMD:R_0603_1608Metric, symbol Device:R
- added R?: 100k, Resistor_SMD:R_0603_1608Metric, symbol Device:R
- C6: value C -> 1nF
- R10, R8, R9: value R -> 1k
- R13: value R -> 150k
- R14: value R -> 10k
- R5: value R -> 329.3k
- R6: value R -> 1.977k
Connections:
- net labels removed: RX_in
- wire segments 132 -> 143
Other:
- moved on the sheet: C7, D?, R11
