File: Light_controller.sch (KiCad schematic (older format))
At the start: 68 parts, among them U1 LM358, U10 PH2.0_horizontal, U11 PH2.0_horizontal, U12 PH2.0_horizontal, U13 PinSocket_1x4, U3 STM8S003F3P, U4 SMD_2062, U5 tact_sw, U6 AMS1117-5.0, U7 EL357N-C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

Commit message: updated schematic for stm8
Parts:
- added C?: 470uF, Capacitor_SMD:CP_Elec_6.3x7.7, symbol Device:C
- added C?: 1nF, Capacitor_SMD:C_0805_2012Metric, symbol Device:C
- added C?: C, Capacitor_SMD:C_0805_2012Metric, symbol Device:C
- added R? (x3): 1.5k, Resistor_SMD:R_0603_1608Metric, symbol Device:R
- added R? (x3): 600, Resistor_SMD:R_0603_1608Metric, symbol Device:R
- added U? (x3): EL357N-C, Package_SO:SOP-4_3.8x4.1mm_P2.54mm, symbol Custom_Library:EL357N-C
- added U?: MAX1487E, symbol Interface_UART:MAX1487E
Connections:
- net labels added: UART_TX_EN
- wire segments 210 -> 256
Other:
- note added: "opto_isolator for UART V1\n"
- note added: "opto_isolator for UART V2\n"
- note added: "opto_isolator for UART V3\n\n"
- note removed: "opto_isolator for UART"
- moved on the sheet: C6, C7, C9, Q?, R10, R8, R9, R?, U10, U7, U8

Commit message: updated schematics for stm8 and esp32
Parts:
- added R32, R34: 600, Resistor_SMD:R_0603_1608Metric, symbol Device:R
- R12: value R -> 22k
- gave numbers to parts that had none: 50
Connections:
- wire segments 256 -> 261
Other:
- note removed: "0.0625 X resistor\n"
- note removed: "18.3K"
- moved on the sheet: C11, C12, C13, D3, R13, R14, R23, R24, R25, R26, R27, R28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
