File: _autosave-Light_controller.sch (KiCad schematic (older format))
At the start: 68 parts, among them U1 LM358, U10 PH2.0_horizontal, U11 PH2.0_horizontal, U12 PH2.0_horizontal, U13 PinSocket_1x4, U3 STM8S003F3P, U4 SMD_2062, U5 tact_sw, U6 AMS1117-5.0, U7 EL357N-C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

Commit message: modified uart circuit for stm8 and stm32
Parts:
- added C?: 470uF, Capacitor_SMD:CP_Elec_6.3x7.7, symbol Device:C
- added C?: 1nF, Capacitor_SMD:C_0805_2012Metric, symbol Device:C
- added C?: C, Capacitor_SMD:C_0805_2012Metric, symbol Device:C
- added R? (x4): 1k, Resistor_SMD:R_0603_1608Metric, symbol Device:R
- added U? (x3): EL357N-C, Package_SO:SOP-4_3.8x4.1mm_P2.54mm, symbol Custom_Library:EL357N-C
- added U?: MAX1487E, symbol Interface_UART:MAX1487E
Connections:
- net labels added: UART_TX_EN
- wire segments 210 -> 253
Other:
- note added: "opto_isolator for UART V1\n"
- note added: "opto_isolator for UART V2\n"
- note added: "opto_isolator for UART V3\n\n"
- note removed: "opto_isolator for UART"
- moved on the sheet: C6, C7, C9, Q?, R10, R8, R9, R?, U10, U7, U8
